File: Kicad/esp32-wled-pcb.kicad_pcb (KiCad board)
At the start: 2 copper layers, 18.7 x 26 mm, 19 parts, among them J1 Conn_01x03_Male, J2 Conn_01x03_Male, J3 SW_Push, J4 SW_Push, Q1 BS170F, U1 ME6211C33M5G, U2 ESP32-PICO-D4

Commit message: intermediate commit
Parts:
- removed J3, J4: SW_Push, Connector_PinHeader_2.54mm:PinHeader_1x02_P2.54mm_Vertical
- added SW1: SW_Push, footprints:SW_XUNPU_TS-1077S, F.Cu at (107.8, 54.6)
- added SW2: SW_Push, footprints:SW_XUNPU_TS-1077S, F.Cu at (107.8, 61.1)
- C1, C2, C3, C4, C5, C6: footprint Capacitor_SMD:C_0805_2012Metric -> Capacitor_SMD:C_0402_1005Metric
- R1, R2, R3, R4, R5: footprint Resistor_SMD:R_0805_2012Metric -> Resistor_SMD:R_0402_1005Metric
- moved Q1 10.8 mm to (118.3, 74.6)
- moved R3 9.22 mm to (121.8, 73.6)
- moved R4 8.78 mm to (123.1, 73.6)
- moved R1 8.65 mm to (113.6, 53.4)
- moved C1 6.98 mm to (109.6, 68.9), turned to 90 degrees
- moved J2 6.94 mm to (116.9, 69.3), turned to 270 degrees
- moved C2 5.87 mm to (113.6, 52.4), turned to 0 degrees
- moved U1 5.59 mm to (107.3, 66.6), turned to 90 degrees
- moved C5 5.25 mm to (106.8, 73.1)
- moved C6 4.45 mm to (110.8, 73.6)
- moved J1 3.75 mm to (124.8, 55.1)
- moved C4 3.32 mm to (115.6, 52.4), turned to 0 degrees
- moved R2 2.82 mm to (111.6, 63.6)
- moved R5 1.74 mm to (110.6, 63.6), turned to 90 degrees
- moved U2 1.18 mm to (114.8, 58.4)
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Routing:
- net +3V3: track 62.0 -> 6.19 mm, vias 6 -> 1
- net GND: track 22.8 -> 1.31 mm, vias 58 -> 1
- net Net-(Q1-Pad3): track 6.35 -> 0.00 mm
- net +5V: track 13.1 -> 7.52 mm
- net /BOOT: track 5.51 -> 0.00 mm
- net Net-(Q1-Pad2): track 4.24 -> 0.00 mm
- net /ESP32_TXD: track 4.18 -> 0.00 mm
- net /LED_DATA: track 3.26 -> 0.00 mm
- net /ESP32_RXD: track 3.14 -> 0.00 mm
- net Net-(AE1-Pad1): track 5.68 -> 4.15 mm
