File: Kicad/esp32-wled-pcb.kicad_pcb (KiCad board)
At the start: 2 copper layers, 18.7 x 26 mm, 19 parts, among them J1 Conn_01x03_Male, J2 Conn_01x03_Male, J3 SW_Push, J4 SW_Push, Q1 BS170F, U1 ME6211C33M5G, U2 ESP32-PICO-D4

Commit message: save in KiCad 6.0 format
Other:
- net class Default removed
