File: Kicad/esp32-wled-pcb.sch (KiCad schematic (older format))
At the start: 26 parts, among them J1 Conn_01x03_Male, J2 Conn_01x03_Male, J3 Conn_01x02_Male, J4 Conn_01x03_Male, J5 Conn_01x02_Male, J6 Conn_01x03_Male, J7 Conn_01x02_Male, J8 Conn_01x02_Male, SW1 SW_Push, SW2 SW_Push, U1 ESP32-PICO-D4, U2 MT3420C

Commit message: still wip
Parts:
- removed J3, J5, J7: Conn_01x02_Male, Connector_JST:JST_PH_B2B-PH-K_1x02_P2.00mm_Vertical, symbol Connector:Conn_01x02_Male
- removed J4, J6: Conn_01x03_Male, Connector_JST:JST_PH_B3B-PH-K_1x03_P2.00mm_Vertical, symbol Connector:Conn_01x03_Male
- added Q1: BS170F, Package_TO_SOT_SMD:SOT-23, symbol Device:Q_NMOS_GSD
- added R5, R7: 4k7, Resistor_SMD:R_0805_2012Metric, symbol Device:R
- added R6: 10k, Resistor_SMD:R_0805_2012Metric, symbol Device:R
- SW1, SW2: footprint (none) -> Button_Switch_SMD:SW_SPST_TL3305B
- renumbered C4 to C1, C5 to C2, C1 to C3, C2 to C4, C3 to C5, C8 to C6, C6 to C7, C7 to C8, J8 to J4, R3 to R2, R4 to R3, R5 to R4, U2 to U1, U1 to U2
Connections:
- net +5V: now also R5.1, R7.1
- net GND: now also R6.2
- net WLED_D1: now also Q1.3 (D), R7.2; no longer U2.16 (IO27)
- net WLED_D2: no longer names the net of U2.14 (IO25)
- net WLED_D3: no longer names the net of U2.15 (IO26)
- new net: Q1.1 (G), R5.2, R6.1
- new net ESP_IO27: Q1.2 (S), U2.16 (IO27)
- no-connect marks 5 -> 31

Commit message: still wip
Parts:
- removed C1, C6, C7: C, Capacitor_SMD:C_0805_2012Metric, symbol Device:C
- removed J4: Conn_01x02_Male, Connector_JST:JST_PH_B2B-PH-K_1x02_P2.00mm_Vertical, symbol Connector:Conn_01x02_Male
- removed L1: L, Inductor_SMD:L_0805_2012Metric, symbol Device:L
- removed R2, R3: R, Resistor_SMD:R_0805_2012Metric, symbol Device:R
- removed U1: MT3420C, Package_TO_SOT_SMD:SOT-23-6, symbol MT3420C:MT3420C
- added C5: 1µ, Capacitor_SMD:C_0805_2012Metric, symbol Device:C
- added R5: 330R, Resistor_SMD:R_0805_2012Metric, symbol Device:R
- added U1: ME6211C33M5G, footprints:SOT95P282X145-5N, symbol ME6211C33M5G:ME6211C33M5G
- C1: renamed from C2; value C -> 1µ
- C2: renamed from C3; value C -> 100n
- C3: renamed from C4; value C -> 10µ
- C4: renamed from C5; value C -> 100n
- C6: renamed from C8; value C -> 10µ
- R4: renamed from R1; value R -> 4k7
- R6: renamed from R4; value R -> 4k7
- SW1, SW2: footprint Button_Switch_SMD:SW_SPST_TL3305B -> footprints:SW_XUNPU_TS-1077S
- renumbered R5 to R1, R6 to R2, R7 to R3
Connections:
- net +3V3: now also C5.1, U1.5 (VOUT)
- net +5V: now also J2.1 (Pin_1), U1.1 (VIN), U1.3 (CE); no longer J2.3 (Pin_3)
- net ESP32_TXD: now also J1.1 (Pin_1); no longer J1.3 (Pin_3)
- net GND: now also J1.3 (Pin_3), J2.3 (Pin_3), C5.2, U1.2 (VSS); no longer J1.1 (Pin_1), J2.1 (Pin_1)
- net ESP_IO27: no longer names the net of U2.16 (IO27)
- net ESP_IO27: now also R5.2; no longer Q1.2 (S)
- net WLED_D1 renamed LED_DATA
- new net: Q1.2 (S), R5.1
Other:
- moved on the sheet: C1, C3, C4, C6, Q1, R1, R2, R3

Commit message: finalize design
Parts:
- removed R1: 4k7, Resistor_SMD:R_0805_2012Metric, symbol Device:R
- removed R5: 330R, Resistor_SMD:R_0805_2012Metric, symbol Device:R
- added R4: 10R, Resistor_SMD:R_0805_2012Metric, symbol Device:R
- J1, J2: footprint Connector_JST:JST_PH_B3B-PH-K_1x03_P2.00mm_Vertical -> Connector_PinHeader_2.54mm:PinHeader_1x03_P2.54mm_Vertical
- J3: renamed from SW1; footprint footprints:SW_XUNPU_TS-1077S -> Connector_PinHeader_2.54mm:PinHeader_1x02_P2.54mm_Vertical; symbol Switch:SW_Push -> Connector:Conn_01x02_Male
- J4: renamed from SW2; footprint footprints:SW_XUNPU_TS-1077S -> Connector_PinHeader_2.54mm:PinHeader_1x02_P2.54mm_Vertical; symbol Switch:SW_Push -> Connector:Conn_01x02_Male
- R2: value 10k -> 4k7
- renumbered R4 to R1, R6 to R5
Connections:
- net +3V3: now also Q1.1 (G), R2.1
- net +5V: now also J2.3 (Pin_3); no longer J2.1 (Pin_1)
- net ESP32_RXD: now also J1.3 (Pin_3); no longer J1.2 (Pin_2)
- net ESP32_TXD: now also J1.2 (Pin_2); no longer J1.1 (Pin_1)
- net GND: now also J1.1 (Pin_1), J2.1 (Pin_1); no longer J1.3 (Pin_3), J2.3 (Pin_3), R2.2
- net LED_DATA: now also R4.1; no longer Q1.3 (D), R3.2
- net at U2.24 (IO4): now also Q1.2 (S), R2.2
- new net: Q1.3 (D), R3.2, R4.2
Other:
- moved on the sheet: Q1, R2, R3

Commit message: intermediate commit
Parts:
- removed J3, J4: SW_Push, Connector_PinHeader_2.54mm:PinHeader_1x02_P2.54mm_Vertical, symbol Connector:Conn_01x02_Male
- added SW1, SW2: SW_Push, footprints:SW_XUNPU_TS-1077S, symbol Switch:SW_Push
- C1, C2, C3, C4, C5, C6: footprint Capacitor_SMD:C_0805_2012Metric -> Capacitor_SMD:C_0402_1005Metric
- R1, R2, R3, R4, R5: footprint Resistor_SMD:R_0805_2012Metric -> Resistor_SMD:R_0402_1005Metric
Connections:
- net BOOT: now also SW2.1
- net GND: now also SW1.1, SW2.2
- net RST: now also SW1.2
Changed lines of the file:
@@
 F 0 "R1" H 3550 1950 50  0000 L CNN
 F 1 "4k7" V 3500 1950 50  0000 C CNN
-F 2 "Resistor_SMD:R_0805_2012Metric" V 3430 1950 50  0001 C CNN
+F 2 "Resistor_SMD:R_0402_1005Metric" V 3430 1950 50  0001 C CNN
 F 3 "~" H 3500 1950 50  0001 C CNN
 	1    3500 1950
@@
 F 0 "C2" H 3550 2500 50  0000 L CNN
 F 1 "100n" H 3550 2300 50  0000 L CNN
-F 2 "Capacitor_SMD:C_0805_2012Metric" H 3538 2250 50  0001 C CNN
+F 2 "Capacitor_SMD:C_0402_1005Metric" H 3538 2250 50  0001 C CNN
 F 3 "~" H 3500 2400 50  0001 C CNN
 	1    3500 2400
@@
 F 0 "C1" H 3250 6700 50  0000 L CNN
 F 1 "1µ" H 3250 6500 50  0000 L CNN
-F 2 "Capacitor_SMD:C_0805_2012Metric" H 3238 6450 50  0001 C CNN
+F 2 "Capacitor_SMD:C_0402_1005Metric" H 3238 6450 50  0001 C CNN
 F 3 "~" H 3200 6600 50  0001 C CNN
 	1    3200 6600
@@
 F 0 "C6" H 5600 6700 50  0000 L CNN
 F 1 "10µ" H 5600 6500 50  0000 L CNN
-F 2 "Capacitor_SMD:C_0805_2012Metric" H 5588 6450 50  0001 C CNN
+F 2 "Capacitor_SMD:C_0402_1005Metric" H 5588 6450 50  0001 C CNN
 F 3 "~" H 5550 6600 50  0001 C CNN
 	1    5550 6600
@@
 Wire Wire Line
 	4950 5150 4950 5200
-$Comp
-L Connector:Conn_01x02_Male J3
-U 1 1 6162BCB9
-P 3000 2250
-F 0 "J3" H 2900 2200 50  0000 C CNN
-F 1 "SW_Push" V 2850 2450 50  0001 C CNN
-F 2 "Connector_PinHeader_2.54mm:PinHeader_1x02_P2.54mm_Vertical" H 3000 2450 50  0001 C CNN
-F 3 "~" H 3000 2450 50  0001 C CNN
-	1    3000 2250
-	1    0    0    1
-$EndComp
 Wire Wire Line
 	3500 2150 3500 2250
 Wire Wire Line
 	3500 2550 3500 2650
-Wire Wire Line
-	3500 2650 3300 2650
-Wire Wire Line
-	3300 2650 3300 2250
 $Comp
 L power:GND #PWR09
@@
 F 0 "C4" H 4450 1600 50  0000 L CNN
 F 1 "100n" H 4450 1400 50  0000 L CNN
-F 2 "Capacitor_SMD:C_0805_2012Metric" H 4438 1350 50  0001 C CNN
+F 2 "Capacitor_SMD:C_0402_1005Metric" H 4438 1350 50  0001 C CNN
 F 3 "~" H 4400 1500 50  0001 C CNN
 	1    4400 1500
@@
 F 0 "C3" H 4050 1600 50  0000 L CNN
 F 1 "10µ" H 4050 1400 50  0000 L CNN
-F 2 "Capacitor_SMD:C_0805_2012Metric" H 4038 1350 50  0001 C CNN
+F 2 "Capacitor_SMD:C_0402_1005Metric" H 4038 1350 50  0001 C CNN
 F 3 "~" H 4000 1500 50  0001 C CNN
 	1    4000 1500
@@
 Wire Wire Line
 	3500 2100 3500 2150
-$Comp
-L Connector:Conn_01x02_Male J4
-U 1 1 616CE137
-P 7750 2450
-F 0 "J4" H 7650 2400 50  0000 C CNN
-F 1 "SW_Push" V 7600 2650 50  0001 C CNN
-F 2 "Connector_PinHeader_2.54mm:PinHeader_1x02_P2.54mm_Vertical" H 7750 2650 50  0001 C CNN
-F 3 "~" H 7750 2650 50  0001 C CNN
-	1    7750 2450
-	-1   0    0    1
-$EndComp
 $Comp
 L Device:R R5
@@
 F 0 "R5" H 7400 2150 50  0000 L CNN
 F 1 "4k7" V 7350 2150 50  0000 C CNN
-F 2 "Resistor_SMD:R_0805_2012Metric" V 7280 2150 50  0001 C CNN
+F 2 "Resistor_SMD:R_0402_1005Metric" V 7280 2150 50  0001 C CNN
 F 3 "~" H 7350 2150 50  0001 C CNN
 	1    7350 2150
@@
 L power:GND #PWR021
 U 1 1 616D049F
-P 7500 2500
-F 0 "#PWR021" H 7500 2250 50  0001 C CNN
-F 1 "GND" H 7505 2327 50  0000 C CNN
-F 2 "" H 7500 2500 50  0001 C CNN
-F 3 "" H 7500 2500 50  0001 C CNN
-	1    7500 2500
+P 7350 2850
+F 0 "#PWR021" H 7350 2600 50  0001 C CNN
+F 1 "GND" H 7355 2677 50  0000 C CNN
+F 2 "" H 7350 2850 50  0001 C CNN
+F 3 "" H 7350 2850 50  0001 C CNN
+	1    7350 2850
 	1    0    0    -1
 $EndComp
@@
 BOOT
 Connection ~ 7350 2350
-Wire Wire Line
-	7350 2350 7550 2350
 Wire Wire Line
 	5750 2350 7350 2350
@@
 F 0 "R2" H 6300 3500 50  0000 L CNN
 F 1 "4k7" V 6250 3500 50  0000 C CNN
-F 2 "Resistor_SMD:R_0805_2012Metric" V 6180 3500 50  0001 C CNN
+F 2 "Resistor_SMD:R_0402_1005Metric" V 6180 3500 50  0001 C CNN
 F 3 "~" H 6250 3500 50  0001 C CNN
 	1    6250 3500
@@
 F 0 "R3" H 6900 3500 50  0000 L CNN
 F 1 "4k7" V 6850 3500 50  0000 C CNN
-F 2 "Resistor_SMD:R_0805_2012Metric" V 6780 3500 50  0001 C CNN
+F 2 "Resistor_SMD:R_0402_1005Metric" V 6780 3500 50  0001 C CNN
 F 3 "~" H 6850 3500 50  0001 C CNN
 	1    6850 3500
@@
 F 0 "C5" H 5200 6700 50  0000 L CNN
 F 1 "1µ" H 5200 6500 50  0000 L CNN
-F 2 "Capacitor_SMD:C_0805_2012Metric" H 5188 6450 50  0001 C CNN
+F 2 "Capacitor_SMD:C_0402_1005Metric" H 5188 6450 50  0001 C CNN
 F 3 "~" H 5150 6600 50  0001 C CNN
 	1    5150 6600
@@
 F 0 "R4" V 7200 3750 50  0000 C CNN
 F 1 "10R" V 7100 3750 50  0000 C CNN
-F 2 "Resistor_SMD:R_0805_2012Metric" V 7030 3750 50  0001 C CNN
+F 2 "Resistor_SMD:R_0402_1005Metric" V 7030 3750 50  0001 C CNN
 F 3 "~" H 7100 3750 50  0001 C CNN
 	1    7100 3750
@@
 	6000 3750 6250 3750
 Connection ~ 6250 3750
+$Comp
+L Switch:SW_Push SW2
+U 1 1 61A1A28B
+P 7350 2600
+F 0 "SW2" V 7304 2748 50  0000 L CNN
+F 1 "SW_Push" V 7395 2748 50  0000 L CNN
+F 2 "footprints:SW_XUNPU_TS-1077S" H 7350 2800 50  0001 C CNN
+F 3 "~" H 7350 2800 50  0001 C CNN
+	1    7350 2600
+	0    1    1    0
+$EndComp
+Wire Wire Line
+	7350 2350 7350 2400
+$Comp
+L Switch:SW_Push SW1
+U 1 1 61A1DE51
+P 3200 2400
+F 0 "SW1" V 3250 2700 50  0000 R CNN
+F 1 "SW_Push" V 3150 2850 50  0000 R CNN
+F 2 "footprints:SW_XUNPU_TS-1077S" H 3200 2600 50  0001 C CNN
+F 3 "~" H 3200 2600 50  0001 C CNN
+	1    3200 2400
+	0    -1   -1   0
+$EndComp
+Wire Wire Line
+	3200 2150 3200 2200
 Wire Wire Line
 	3200 2150 3500 2150
 Wire Wire Line
-	3300 2250 3200 2250
-Wire Wire Line
-	7550 2450 7500 2450
-Wire Wire Line
-	7500 2450 7500 2500
+	3200 2650 3200 2600
+Wire Wire Line
+	3200 2650 3500 2650
 $EndSCHEMATC
